File: spindle-controller/VFDEnclosure.kicad_sch (KiCad schematic)
At the start: 3 parts, among them J16 Conn_01x11, J23 Conn_01x03, J24 GX12-6

Commit message: Rename project to Spindle_Controller; add VFD_DI1 spindle command path
Renamed CNC_router -> Spindle_Controller for clarity, since this
project is specifically about the spindle controller rather than the
router as a whole. Also adds the GX12-7 cable connector and VFD_DI1
wiring needed to command the spindle on, routes it through a DPDT
safety-interlock switch (SW1) shared with the warning light circuit,
fixes a DAC/ADC signal swap on VFD_VF1/VFD_FM1, and reconciles several
net labels between the root schematic and the VFD Enclosure /
TechnoCNC Controller / Warning Light Box sub-sheets.

Co-Authored-By: Claude Sonnet 5 <noreply@anthropic.com>
Parts:
- J24: value GX12-6 -> GX12-7; symbol Connector:LEMO6 -> GX12_Connectors:GX12-7
Connections:
- net VFD_DI1: now reaches J16.6 (DI1)
- net VFD_DI1: now also J24.7
Changed lines of the file:
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@@
+	(wire
+		(pts
+			(xy 17.78 53.086) (xy 82.804 53.086)
+		)
+		(stroke
+			(width 0)
+			(type default)
+		)
+	)
+	(wire
+		(pts
+			(xy 82.804 49.53) (xy 82.55 49.53)
+		)
+		(stroke
+			(width 0)
+			(type default)
+		)
+	)
 	(wire
 		(pts
@@
 	(wire
 		(pts
-			(xy 110.49 49.53) (xy 110.49 101.6)
-		)
-		(stroke
-			(width 0)
-			(type default)
-		)
-	)
-	(wire
-		(pts
-			(xy 74.93 95.25) (xy 74.93 49.53)
+			(xy 82.804 53.086) (xy 82.804 49.53)
+		)
+		(stroke
+			(width 0)
+			(type default)
+		)
+	)
+	(wire
+		(pts
+			(xy 110.49 49.53) (xy 110.49 113.284)
+		)
+		(stroke
+			(width 0)
+			(type default)
+		)
+	)
+	(wire
+		(pts
+			(xy 31.75 82.55) (xy 17.78 82.55)
+		)
+		(stroke
+			(width 0)
+			(type default)
+		)
+	)
+	(wire
+		(pts
+			(xy 74.676 101.6) (xy 74.676 101.346)
+		)
+		(stroke
+			(width 0)
+			(type default)
+		)
+	)
+	(wire
+		(pts
+			(xy 17.78 82.55) (xy 17.78 53.086)
 		)
 		(stroke
@@
 	(wire
 		(pts
-			(xy 31.75 87.63) (xy 31.75 101.6)
-		)
-		(stroke
-			(width 0)
-			(type default)
-		)
-	)
-	(wire
-		(pts
 			(xy 44.45 69.85) (xy 44.45 60.96)
 		)
@@
 	(wire
 		(pts
+			(xy 31.75 87.63) (xy 31.75 113.284)
+		)
+		(stroke
+			(width 0)
+			(type default)
+		)
+	)
+	(wire
+		(pts
+			(xy 74.93 101.346) (xy 74.93 49.53)
+		)
+		(stroke
+			(width 0)
+			(type default)
+		)
+	)
+	(wire
+		(pts
 			(xy 57.15 77.47) (xy 57.15 38.1)
 		)
@@
 	(wire
 		(pts
+			(xy 74.676 101.346) (xy 74.93 101.346)
+		)
+		(stroke
+			(width 0)
+			(type default)
+		)
+	)
+	(wire
+		(pts
 			(xy 57.15 87.63) (xy 60.96 87.63)
 		)
@@
 	(wire
 		(pts
-			(xy 31.75 101.6) (xy 110.49 101.6)
-		)
-		(stroke
-			(width 0)
-			(type default)
-		)
-	)
-	(wire
-		(pts
-			(xy 44.45 95.25) (xy 74.93 95.25)
+			(xy 31.75 113.284) (xy 110.49 113.284)
+		)
+		(stroke
+			(width 0)
+			(type default)
+		)
+	)
+	(wire
+		(pts
+			(xy 44.196 101.6) (xy 74.676 101.6)
+		)
+		(stroke
+			(width 0)
+			(type default)
+		)
+	)
+	(wire
+		(pts
+			(xy 44.196 101.6) (xy 44.45 95.25)
 		)
 		(stroke
@@
 	(global_label "VFD_RUN_SENSE"
 		(shape output)
-		(at 31.75 101.6 180)
+		(at 31.75 101.346 180)
 		(fields_autoplaced yes)
 		(effects
@@
 		)
 		(property "Intersheetrefs" "${INTERSHEET_REFS}"
-			(at 13.4039 101.6 0)
+			(at 13.4039 101.346 0)
 			(hide yes)
 			(show_name no)
@@
 		)
 	)
-	(global_label "VFD_FM1"
-		(shape output)
-		(at 45.72 95.25 180)
+	(global_label "VFD_DI1"
+		(shape input)
+		(at 22.098 82.55 270)
 		(fields_autoplaced yes)
 		(effects
 			(font
 				(size 1.27 1.27)
+				(thickness 0.254)
+				(bold yes)
 			)
 			(justify right)
 		)
 		(property "Intersheetrefs" "${INTERSHEET_REFS}"
-			(at 34.5705 95.25 0)
+			(at 22.098 93.5103 90)
 			(hide yes)
 			(show_name no)
@@
 		)
 	)
+	(global_label "VFD_FM1"
+		(shape output)
+		(at 45.466 101.6 180)
+		(fields_autoplaced yes)
+		(effects
+			(font
+				(size 1.27 1.27)
+			)
+			(justify right)
+		)
+		(property "Intersheetrefs" "${INTERSHEET_REFS}"
+			(at 34.3165 101.6 0)
+			(hide yes)
+			(show_name no)
+			(do_not_autoplace no)
+			(effects
+				(font
+					(size 1.27 1.27)
+				)
+				(justify right)
+			)
+		)
+	)
 	(symbol
-		(lib_id "Connector:LEMO6")
+		(lib_id "GX12_Connectors:GX12-7")
 		(at 44.45 82.55 0)
 		(unit 1)
@@
 			)
 		)
-		(property "Value" "GX12-6"
+		(property "Value" "GX12-7"
 			(at 46.1011 69.85 0)
 			(show_name no)
@@
 			)
 		)
-		(property "Description" "6-pin LEMO connector"
+		(property "Description" "7-pin GX12 Connector"
 			(at 44.45 82.55 0)
 			(hide yes)
@@
 		(pin "1"
 		)
+		(pin "7"
+		)
 		(instances
-			(project "CNC_router"
+			(project "Spindle_Controller"
 				(path "/10c7a81d-d8e0-4023-94dc-af5199d847de/f7b14e96-f363-41c6-90b3-9bd94a39e254"
 					(reference "J24")
@@
 		)
 		(instances
-			(project "CNC_router"
+			(project "Spindle_Controller"
 				(path "/10c7a81d-d8e0-4023-94dc-af5199d847de/f7b14e96-f363-41c6-90b3-9bd94a39e254"
 					(reference "J16")
@@
 		)
 		(instances
-			(project "CNC_router"
+			(project "Spindle_Controller"
 				(path "/10c7a81d-d8e0-4023-94dc-af5199d847de/f7b14e96-f363-41c6-90b3-9bd94a39e254"
 					(reference "J23")
