File: spindle-controller/VFDEnclosure.kicad_sch (KiCad schematic)
At the start: 3 parts, among them J16 Conn_01x11, J23 Conn_01x03, J24 GX12-7

Commit message: updated connectors
Connections:
- no-connect marks 0 -> 1
Other:
- note added: "FM1 -- analog output, actual running frequency (0-10V, shares GND below) Requires P2.0.33 = 00 (Run frequency) This is already the Factory default Requires J6 in 0-10V"
- note removed: "FM1 -- analog output, actual running frequency (0-10V, shares GND below) Requires P2.0.33 = 00 (Run frequency) This is already the Factory default Requires J6 in 0-10V position"
Changed lines of the file:
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@@
+		)
+	)
+	(circle
+		(center 44.45 82.042)
+		(radius 0.508)
+		(stroke
+			(width 0)
+			(type solid)
+			(color 132 0 0 1)
+		)
+		(fill
+			(type none)
 		)
 	)
@@
 		)
 	)
-	(text "FM1 -- analog output, actual running frequency\n(0-10V, shares GND below)\nRequires P2.0.33 = 00 (Run frequency)\n	This is already the Factory default\nRequires J6 in 0-10V position"
+	(text "FM1 -- analog output, actual running frequency\n(0-10V, shares GND below)\nRequires P2.0.33 = 00 (Run frequency)\n	This is already the Factory default\nRequires J6 in 0-10V "
 		(exclude_from_sim no)
 		(at 125.73 50.8 0)
@@
 		(diameter 0)
 		(color 0 0 0 0)
+	)
+	(no_connect
+		(at 115.57 49.53)
 	)
 	(wire
@@
 		)
 	)
+	(polyline
+		(pts
+			(xy 34.29 82.55) (xy 44.196 82.55)
+		)
+		(stroke
+			(width 0)
+			(type default)
+		)
+	)
 	(wire
 		(pts
@@
 		)
 		(stroke
+			(width 0)
+			(type default)
+		)
+	)
+	(polyline
+		(pts
+			(xy 44.196 82.55) (xy 44.196 82.804)
+		)
+		(stroke
