File: spindle-controller/Spindle_Controller.kicad_sch (KiCad schematic)
At the start: 25 parts, among them J1 Conn_01x19, J10 Conn_01x03, J11 Conn_01x02, J12 Conn_01x04, J13 Conn_01x02, J14 Conn_01x04, J18 GX16-8, J19 GX12-4, J2 Conn_01x19, J20 DIN-3, J21 DIN-3, J26 GX12-2, J27 GX12-2, J3 Conn_01x14, J4 Jack-DC, J5 USB_C_Receptacle_USB2.0_16P, J6 Conn_01x04, J7 Conn_01x04, J8 Conn_01x04, J9 Conn_01x05, K2 JQC-3FF-005-1Z, K3 JQC-3FF-005-1Z, K4 JQC-3FF-005-1Z, K5 JQC-3FF-005-1Z, SW1 DPDT Toggle Switch

Commit message: fixed schematics
Parts:
- removed J27: GX12-2, symbol Connector:LEMO2
- added J15: GX12-3, symbol Connector:DIN-3
Connections:
- net at K2.11: now also J15.3
- net at K2.14: now also J15.1
- no-connect marks 21 -> 22
Changed lines of the file:
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@@
 		)
 	)
-	(text "Relay #3"
+	(text "Relay #4"
 		(exclude_from_sim no)
 		(at 116.332 86.106 0)
@@
 	)
 	(no_connect
+		(at 186.69 172.72)
+	)
+	(no_connect
 		(at 135.89 228.6)
 	)
@@
 	(wire
 		(pts
+			(xy 194.31 180.34) (xy 194.31 190.5)
+		)
+		(stroke
+			(width 0)
+			(type default)
+		)
+	)
+	(wire
+		(pts
 			(xy 92.71 163.83) (xy 125.73 163.83)
 		)
@@
 	(wire
 		(pts
-			(xy 176.53 190.5) (xy 213.36 190.5)
+			(xy 58.42 40.64) (xy 72.39 40.64)
 		)
 		(stroke
@@
 	(wire
 		(pts
-			(xy 58.42 40.64) (xy 72.39 40.64)
+			(xy 179.07 167.64) (xy 215.9 167.64)
 		)
 		(stroke
@@
 		)
 	)
-	(wire
-		(pts
-			(xy 176.53 167.64) (xy 215.9 167.64)
-		)
-		(stroke
-			(width 0)
-			(type default)
-		)
-	)
 	(polyline
 		(pts
@@
 	(wire
 		(pts
-			(xy 176.53 182.88) (xy 176.53 190.5)
+			(xy 179.07 180.34) (xy 179.07 167.64)
 		)
 		(stroke
@@
 	(wire
 		(pts
-			(xy 176.53 180.34) (xy 176.53 167.64)
-		)
-		(stroke
-			(width 0)
-			(type default)
-		)
-	)
-	(wire
-		(pts
 			(xy 254 23.591) (xy 254 31.75)
 		)
@@
 	(wire
 		(pts
+			(xy 194.31 190.5) (xy 213.36 190.5)
+		)
+		(stroke
+			(width 0)
+			(type default)
+		)
+	)
+	(wire
+		(pts
 			(xy 173.99 33.02) (xy 173.99 148.59)
 		)
@@
 	)
 	(symbol
-		(lib_id "Connector:LEMO2")
-		(at 184.15 180.34 0)
-		(mirror x)
-		(unit 1)
-		(body_style 1)
-		(exclude_from_sim no)
-		(in_bom yes)
-		(on_board yes)
-		(in_pos_files yes)
-		(dnp no)
-		(property "Reference" "J27"
-			(at 188.976 182.8801 0)
-			(hide yes)
-			(show_name no)
-			(do_not_autoplace no)
-			(effects
-				(font
-					(size 1.27 1.27)
-				)
-				(justify left)
-			)
-		)
-		(property "Value" "GX12-2"
-			(at 183.5785 175.26 0)
-			(show_name no)
-			(do_not_autoplace no)
-			(effects
-				(font
-					(size 1.27 1.27)
-				)
-			)
-		)
-		(property "Footprint" ""
-			(at 184.15 181.61 0)
-			(hide yes)
-			(show_name no)
-			(do_not_autoplace no)
-			(effects
-				(font
-					(size 1.27 1.27)
-				)
-			)
-		)
-		(property "Datasheet" ""
-			(at 184.15 181.61 0)
-			(hide yes)
-			(show_name no)
-			(do_not_autoplace no)
-			(effects
-				(font
-					(size 1.27 1.27)
-				)
-			)
-		)
-		(property "Description" "2-pin LEMO connector"
-			(at 184.15 180.34 0)
-			(hide yes)
-			(show_name no)
-			(do_not_autoplace no)
-			(effects
-				(font
-					(size 1.27 1.27)
-				)
-			)
-		)
-		(pin "2"
-		)
-		(pin "1"
-		)
-		(instances
-			(project "Spindle_Controller"
-				(path "/10c7a81d-d8e0-4023-94dc-af5199d847de"
-					(reference "J27")
-					(unit 1)
-				)
-			)
-		)
-	)
-	(symbol
 		(lib_name "Conn_01x04_1")
 		(lib_id "Connector_Generic:Conn_01x04")
@@
 					(unit 1)
 				)
+			)
+		)
+	)
+	(symbol
+		(lib_id "Connector:DIN-3")
+		(at 186.69 180.34 0)
+		(unit 1)
+		(body_style 1)
+		(exclude_from_sim no)
+		(in_bom yes)
+		(on_board yes)
+		(in_pos_files yes)
+		(dnp no)
+		(property "Reference" "J15"
+			(at 186.69 187.96 0)
+			(show_name no)
+			(do_not_autoplace no)
+			(effects
+				(font
+					(size 1.27 1.27)
+				)
+			)
+		)
+		(property "Value" "GX12-3"
+			(at 186.944 169.672 0)
+			(show_name no)
+			(do_not_autoplace no)
+			(effects
+				(font
+					(size 1.27 1.27)
+				)
+			)
+		)
+		(property "Footprint" ""
+			(at 186.69 180.34 0)
+			(hide yes)
+			(show_name no)
+			(do_not_autoplace no)
+			(effects
+				(font
+					(size 1.27 1.27)
+				)
+			)
+		)
+		(property "Datasheet" "http://www.mouser.com/ds/2/18/40_c091_abd_e-75918.pdf"
+			(at 186.69 180.34 0)
+			(hide yes)
+			(show_name no)
+			(do_not_autoplace no)
+			(effects
+				(font
+					(size 1.27 1.27)
+				)
+			)
+		)
+		(property "Description" "3-pin DIN connector"
+			(at 186.69 180.34 0)
+			(hide yes)
+			(show_name no)
+			(do_not_autoplace no)
+			(effects
+				(font
+					(size 1.27 1.27)
+				)
+			)
+		)
+		(pin "1"
+		)
+		(pin "2"
+		)
+		(pin "3"
+		)
+		(instances
+			(project "Spindle_Controller"
+				(path "/10c7a81d-d8e0-4023-94dc-af5199d847de"
+					(reference "J15")
+					(unit 1)
+				)

Commit message: changes to control box and pendant project
Other:
- note added: "NB: All colors correspond to colors in the enclosure and NOT the cables"
Changed lines of the file:
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@@
+		)
+	)
+	(text "NB: All colors correspond to colors in the enclosure and NOT the cables"
+		(exclude_from_sim no)
+		(at 197.612 276.098 0)
+		(effects
+			(font
+				(face "KiCad Font")
+				(size 2.54 2.54)
+				(thickness 0.508)
+				(bold yes)
+			)
 		)
 	)
@@
 	(text "Orange Wire"
 		(exclude_from_sim no)
-		(at 226.06 248.92 0)
+		(at 232.41 238.252 0)
 		(effects
 			(font
@@
 	(text "White Wire"
 		(exclude_from_sim no)
-		(at 229.87 232.41 0)
+		(at 227.584 248.412 0)
 		(effects
 			(font
