File: spindle-controller/OriginalSpindleController.kicad_sch (KiCad schematic)
At the start: 9 parts, among them J29 GX12-6, J30 GX12-2, J31 GX16-8, J32 GX12-6, J33 GX16-8, J35 Conn_01x11, J36 Conn_01x03, J37 GX12-4, SW2 DPDT Switch

Commit message: changes to control box and pendant project
Parts:
- added SW3: SW_SPST, Button_Switch_THT:SW_NKK_NR01, symbol Switch:SW_SPST
Connections:
- net VFD_24V: now also J35.10 (OP)
- net VFD_COM: now also J36.1 (TA), SW3.2 (B)
- net VFD_GND: no longer J36.1 (TA)
- net at J35.9 (DI4): now also SW3.1 (A)
- no-connect marks 8 -> 6
Other:
- note added: "Keyed Switch"
- note added: "N.B: Logic Signals must be relative to COM and NOT GND. - GND is power ground - COM is logic ground GND and COMM are isolated from one another, but there are sneak paths between them. OP tied to +24 will allow DIx to be active if tied to COM OP tied to COM will allow DIx to be active if tied to +24V. [NOT IN MANUAL]"
- note added: "SW3 is a keyed switch that when on (green) enables the "standard" control know to set the frequency. when it is off (red), the "keypad" is ignored and VF1 signal sets the frequency (external source)"
Changed lines of the file:
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@@
+		)
+	)
+	(text "N.B:    Logic Signals must be relative to \nCOM and NOT GND.\n-                       GND is power ground\n-                       COM is logic ground\nGND and COMM are isolated from one another, but there are \nsneak paths between them.\n\nOP tied to +24 will allow DIx to be active if tied to COM\nOP tied to COM will allow DIx to be active if tied to +24V.\n[NOT IN MANUAL]"
+		(exclude_from_sim no)
+		(at 317.754 69.85 0)
+		(effects
+			(font
+				(size 1.27 1.27)
+			)
 		)
 	)
@@
 		)
 	)
+	(text "Keyed Switch"
+		(exclude_from_sim no)
+		(at 217.17 51.562 0)
+		(effects
+			(font
+				(size 1.27 1.27)
+			)
+		)
+	)
+	(text "SW3 is a keyed switch that when on (green)\nenables the \"standard\" control know to set\nthe frequency.\n\nwhen it is off (red), the \"keypad\"  is ignored and VF1 signal \nsets the frequency (external source)"
+		(exclude_from_sim no)
+		(at 291.084 91.948 0)
+		(effects
+			(font
+				(size 1.27 1.27)
+			)
+			(justify left)
+		)
+	)
 	(text "Original Spindle Controller"
 		(exclude_from_sim no)
@@
 	)
 	(junction
-		(at 232.41 49.53)
+		(at 250.19 48.26)
 		(diameter 0)
 		(color 0 0 0 0)
 	)
+	(junction
+		(at 234.95 49.53)
+		(diameter 0)
+		(color 0 0 0 0)
+	)
 	(no_connect
 		(at 240.03 45.72)
@@
 	)
 	(no_connect
-		(at 245.11 45.72)
-	)
-	(no_connect
-		(at 247.65 45.72)
-	)
-	(no_connect
 		(at 62.23 55.88)
 	)
@@
 	(wire
 		(pts
-			(xy 265.43 49.53) (xy 232.41 49.53)
-		)
-		(stroke
-			(width 0)
-			(type default)
-		)
-	)
-	(wire
-		(pts
 			(xy 20.32 92.71) (xy 20.32 116.84)
 		)
@@
 	(wire
 		(pts
+			(xy 212.09 38.1) (xy 256.54 38.1)
+		)
+		(stroke
+			(width 0)
+			(type default)
+		)
+	)
+	(wire
+		(pts
+			(xy 247.65 48.26) (xy 250.19 48.26)
+		)
+		(stroke
+			(width 0)
+			(type default)
+		)
+	)
+	(wire
+		(pts
 			(xy 237.49 45.72) (xy 237.49 58.42)
 		)
@@
 	(wire
 		(pts
+			(xy 247.65 45.72) (xy 247.65 48.26)
+		)
+		(stroke
+			(width 0)
+			(type default)
+		)
+	)
+	(wire
+		(pts
 			(xy 120.65 93.98) (xy 142.24 93.98)
 		)
@@
 	(wire
 		(pts
+			(xy 212.09 48.26) (xy 212.09 38.1)
+		)
+		(stroke
+			(width 0)
+			(type default)
+		)
+	)
+	(wire
+		(pts
 			(xy 257.81 107.95) (xy 260.35 107.95)
 		)
@@
 	(wire
 		(pts
+			(xy 234.95 45.72) (xy 234.95 49.53)
+		)
+		(stroke
+			(width 0)
+			(type default)
+		)
+	)
+	(wire
+		(pts
 			(xy 130.81 76.2) (xy 138.43 76.2)
 		)
@@
 	(wire
 		(pts
+			(xy 245.11 46.99) (xy 245.11 45.72)
+		)
+		(stroke
+			(width 0)
+			(type default)
+		)
+	)
+	(wire
+		(pts
 			(xy 219.71 107.95) (xy 227.33 107.95)
 		)
@@
 	(wire
 		(pts
+			(xy 256.54 38.1) (xy 256.54 46.99)
+		)
+		(stroke
+			(width 0)
+			(type default)
+		)
+	)
+	(wire
+		(pts
 			(xy 242.57 59.69) (xy 242.57 92.71)
 		)
@@
 	(wire
 		(pts
+			(xy 256.54 46.99) (xy 245.11 46.99)
+		)
+		(stroke
+			(width 0)
+			(type default)
+		)
+	)
+	(wire
+		(pts
 			(xy 237.49 58.42) (xy 219.71 58.42)
 		)
@@
 	(wire
 		(pts
-			(xy 232.41 49.53) (xy 232.41 50.8)
+			(xy 222.25 49.53) (xy 234.95 49.53)
 		)
 		(stroke
@@
 	(wire
 		(pts
-			(xy 232.41 45.72) (xy 232.41 49.53)
+			(xy 232.41 45.72) (xy 232.41 50.8)
 		)
 		(stroke
@@
 	(wire
 		(pts
+			(xy 234.95 49.53) (xy 234.95 57.15)
+		)
+		(stroke
+			(width 0)
+			(type default)
+		)
+	)
+	(wire
+		(pts
+			(xy 222.25 49.53) (xy 222.25 48.26)
+		)
+		(stroke
+			(width 0)
+			(type default)
+		)
+	)
+	(wire
+		(pts
+			(xy 234.95 49.53) (xy 265.43 49.53)
+		)
+		(stroke
+			(width 0)
+			(type default)
+		)
+	)
+	(wire
+		(pts
 			(xy 96.52 106.68) (xy 107.95 106.68)
 		)
@@
 	(wire
 		(pts
-			(xy 234.95 45.72) (xy 234.95 57.15)
-		)
-		(stroke
-			(width 0)
-			(type default)
-		)
-	)
-	(wire
-		(pts
 			(xy 265.43 46.99) (xy 265.43 49.53)
 		)
@@
 			)
 		)
+	)
+	(symbol
+		(lib_id "Switch:SW_SPST")
+		(at 217.17 48.26 0)
+		(unit 1)
+		(body_style 1)
+		(exclude_from_sim no)
+		(in_bom yes)
+		(on_board yes)
+		(in_pos_files yes)
+		(dnp no)
+		(fields_autoplaced yes)
+		(property "Reference" "SW3"
+			(at 217.17 41.91 0)
+			(show_name no)
+			(do_not_autoplace no)
+			(effects
+				(font
+					(size 1.27 1.27)
+				)
+			)
+		)
+		(property "Value" "SW_SPST"
+			(at 217.17 44.45 0)
+			(show_name no)
+			(do_not_autoplace no)
+			(effects
+				(font
+					(size 1.27 1.27)
+				)
+			)
+		)
+		(property "Footprint" "Button_Switch_THT:SW_NKK_NR01"
+			(at 217.17 48.26 0)
+			(hide yes)
+			(show_name no)
+			(do_not_autoplace no)
+			(effects
+				(font
+					(size 1.27 1.27)
+				)
+			)
+		)
+		(property "Datasheet" ""
+			(at 217.17 48.26 0)
+			(hide yes)
+			(show_name no)
+			(do_not_autoplace no)
+			(effects
+				(font
+					(size 1.27 1.27)
+				)
+			)
+		)
+		(property "Description" "Single Pole Single Throw (SPST) switch"
+			(at 217.17 48.26 0)
+			(hide yes)
+			(show_name no)
+			(do_not_autoplace no)
+			(effects
+				(font
+					(size 1.27 1.27)
+				)
+			)
+		)
+		(pin "2"
+		)
+		(pin "1"
+		)
+		(instances
+			(project "Spindle_Controller"
+				(path "/10c7a81d-d8e0-4023-94dc-af5199d847de/b4e88c76-d553-44d8-aeeb-aa4b7ae1f43a"
+					(reference "SW3")
+					(unit 1)
+				)
+			)
+		)

Commit message: OriginalSpindleController: fix typos in SW3 and COM/GND notes
Other:
- note added: "N.B: Logic Signals must be relative to COM and NOT GND. - GND is power ground - COM is logic ground GND and COM are isolated from one another, but there are sneak paths between them. OP tied to +24 will allow DIx to be active if tied to COM OP tied to COM will allow DIx to be active if tied to +24V. [NOT IN MANUAL]"
- note added: "SW3 is a keyed switch that when on (green) enables the "standard" control knob to set the frequency. when it is off (red), the "keypad" is ignored and VF1 signal sets the frequency (external source)"
- note removed: "N.B: Logic Signals must be relative to COM and NOT GND. - GND is power ground - COM is logic ground GND and COMM are isolated from one another, but there are sneak paths between them. OP tied to +24 will allow DIx to be active if tied to COM OP tied to COM will allow DIx to be active if tied to +24V. [NOT IN MANUAL]"
- note removed: "SW3 is a keyed switch that when on (green) enables the "standard" control know to set the frequency. when it is off (red), the "keypad" is ignored and VF1 signal sets the frequency (external source)"
Changed lines of the file:
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@@
 		)
 	)
-	(text "N.B:    Logic Signals must be relative to \nCOM and NOT GND.\n-                       GND is power ground\n-                       COM is logic ground\nGND and COMM are isolated from one another, but there are \nsneak paths between them.\n\nOP tied to +24 will allow DIx to be active if tied to COM\nOP tied to COM will allow DIx to be active if tied to +24V.\n[NOT IN MANUAL]"
+	(text "N.B:    Logic Signals must be relative to \nCOM and NOT GND.\n-                       GND is power ground\n-                       COM is logic ground\nGND and COM are isolated from one another, but there are \nsneak paths between them.\n\nOP tied to +24 will allow DIx to be active if tied to COM\nOP tied to COM will allow DIx to be active if tied to +24V.\n[NOT IN MANUAL]"
 		(exclude_from_sim no)
 		(at 317.754 69.85 0)
@@
 		)
 	)
-	(text "SW3 is a keyed switch that when on (green)\nenables the \"standard\" control know to set\nthe frequency.\n\nwhen it is off (red), the \"keypad\"  is ignored and VF1 signal \nsets the frequency (external source)"
+	(text "SW3 is a keyed switch that when on (green)\nenables the \"standard\" control knob to set\nthe frequency.\n\nwhen it is off (red), the \"keypad\"  is ignored and VF1 signal \nsets the frequency (external source)"
 		(exclude_from_sim no)
 		(at 291.084 91.948 0)
