File: spindle-controller/SpindleProbe/SpindleProbe.kicad_sch (KiCad schematic)
At the start: 20 parts, among them SW1 SPST Tilt Switch, U1 LM741, U2 DRV5055A1xDBZxQ1

Commit message: changes to control box and pendant project
Parts:
- added J1: DIN-4, Display:CR2013-MI2120, symbol Connector:DIN-4
- added J2: LEMO2, Display:CR2013-MI2120, symbol Connector:LEMO2
Connections:
- new net: J1.4, J2.1
Other:
- note added: "GX12-2"
- note added: "GX12-4"
- note added: "Green ANODE"
- note added: "Green on Cable to probe"
- note added: "Hall Probe GND Black Wire"
- note added: "Hall Probe Output Blue Wire"
- note added: "Hall Probe Vcc Red Wire"
- note added: "Red Anode"
- note added: "Touch Probe Contact Yellow Wire"
- note added: "Touch Probe Plate"
- note removed: "Green Anode"
- note removed: "Red ANODE"
